Commit message: fix base box not anchored to the ground

File: single_lwr_example/single_lwr_robot/robot/single_lwr_robot.urdf.xacro (robot description, xacro)
@@ -29,4 +29,10 @@
 		<static>true</static>>
 	</gazebo>
+	<link name="world" />
+	<joint name="world_joint"  type="fixed">
+	  <origin xyz="0 0 0" rpy="0 0 0" />
+	  <parent link="world"/>
+	  <child link="box"/>
+	</joint>
 	<!-- using the models -->
 	<xacro:kuka_lwr parent="box" name="lwr">

Commit message: -change robot base size -add workspace box

File: single_lwr_example/single_lwr_robot/robot/single_lwr_robot.urdf.xacro (robot description, xacro)
@@ -5,5 +5,5 @@
 	<!-- and assemble your robot -->
 	<link name="box">
-		<inertial>
+	  <inertial>
 			<mass value="5.0"/>
 			<origin rpy="0 0 0" xyz="0 0 0"/>
@@ -14,13 +14,13 @@
 		</inertial>
 		<visual>
-			<origin xyz="0 0 0.50" rpy="0 0 0"/>
+		  <origin xyz="0 0 0.5" rpy="0 0 0"/>
 			<geometry>
-				<box size="1.0 1.0 1.0"/>
+			  <box size="0.5 0.5 1"/>
 			</geometry>
 		</visual>
 		<collision>
-			<origin xyz="0 0 0.50" rpy="0 0 0"/>
+			<origin xyz="0 0 0.5" rpy="0 0 0"/>
 			<geometry>
-				<box size="1.0 1.0 1.0"/>
+			  <box size="0.5 0.5 1"/>
 			</geometry>
 		</collision>
@@ -31,5 +31,4 @@
 	<link name="world" />
 	<joint name="world_joint"  type="fixed">
-	  <origin xyz="0 0 0" rpy="0 0 0" />
 	  <parent link="world"/>
 	  <child link="box"/>
