Commit message: -add force torque sensor -add a dummy link and joint required by the sensor

File: lwr_description/model/kuka_lwr.gazebo.xacro (robot description, xacro)
@@ -6,4 +6,11 @@
 				<robotNamespace>${name}</robotNamespace>
 			</plugin>
+		</gazebo>
+		<gazebo>
+		  <plugin name="FTsensor_controller" filename="libgazebo_ros_ft_sensor.so">
+		    <updateRate>100.0</updateRate>
+		    <topicName>${name}/ft_sensor</topicName>
+		    <jointName>sensor_joint</jointName>
+		  </plugin>
 		</gazebo>
 		<gazebo reference="${name}_base_link">
@@ -39,4 +46,12 @@
 			<material>Gazebo/Grey</material>
 		</gazebo>
+		<gazebo reference="end_effector">
+			<gravity>true</gravity>
+			<material>Gazebo/Red</material>
+		</gazebo>
+		<gazebo reference="sensor_joint">
+		  <provideFeedback>true</provideFeedback>
+		  <disableFixedJointLumping>true</disableFixedJointLumping>
+		</gazebo>
 	</xacro:macro>
 </robot>

File: lwr_description/model/kuka_lwr.urdf.xacro (robot description, xacro)
@@ -11,6 +11,6 @@
 	<xacro:property name="base_mass" value="2.0"/>
 	<xacro:property name="link_mass" value="2.35"/>
-    <xacro:property name="wrist_mass" value="1.1"/>
-    <xacro:property name="tip_mass" value="0.25"/>
+	<xacro:property name="wrist_mass" value="1.1"/>
+	<xacro:property name="tip_mass" value="0.25"/>
 	<xacro:property name="velocity_scale" value="1"/>
 	<xacro:property name="effort_scale" value="1"/>
@@ -359,8 +359,33 @@
 			<material name="Kuka/DarkGrey"/>
 			</visual>
-			<collision>
-			<origin xyz="0 0 0" rpy="0 0 ${M_PI}"/>
+			<!-- <collision> -->
+			<!-- <origin xyz="0 0 0" rpy="0 0 ${M_PI}"/> -->
+			<!-- <geometry> -->
+			<!-- 	<cylinder radius="0.04" length="0.015"/> -->
+			<!-- </geometry> -->
+			<!-- </collision> -->
+		</link>
+		<joint name="sensor_joint" type="fixed">
+			<origin xyz="0 0 0.005" rpy="0 0 0"/>
+			<parent link="${name}_7_link"/>
+			<child link="end_effector"/>
+		</joint>
+		<link name="end_effector">
+			<inertial>
+				<mass value="0.1"/>
+				<origin xyz="0 0 0"/>
+				<cylinder_inertia_def radius="0.03" length="0.01" mass="0.1"/>
+			</inertial>
+			<visual>
+				<origin xyz="0 0 0" rpy="0 0 0"/>
+				<geometry>
+				  <cylinder radius="0.03" length="0.01"/>
+				</geometry>
+			<material name="Black"/>
+			</visual>
+			<collision>
+			<origin xyz="0 0 0" rpy="0 0 0"/>
 			<geometry>
-				<cylinder radius="0.04" length="0.05"/>
+				<cylinder radius="0.03" length="0.01"/>
 			</geometry>
 			</collision>
