Commit message: playing around with extra joints and handles to use position_controllers/JointTrajectoryController for handling position, stiffness, damping, and additional torque for the kuka arm

File: lwr_description/model/kuka_lwr.urdf.xacro (robot description, xacro)
@@ -18,4 +18,10 @@
 	<xacro:property name="min_stiffness" value="0"/>
 	<xacro:property name="rate_stiffness" value="20000"/> <!-- reflex to stiffness -->
+	<xacro:property name="max_damping" value="1.0"/>
+	<xacro:property name="min_damping" value="0.0"/>
+	<xacro:property name="rate_damping" value="4.0"/> <!-- reflex to damping -->
+	<xacro:property name="max_add_torque" value="-1.0"/>
+	<xacro:property name="min_add_torque" value="1.0"/>
+	<xacro:property name="rate_add_torque" value="8.0"/> <!-- reflex to additional torque -->
 	<!-- URDF model /-->
 	<xacro:macro name="kuka_lwr" params="parent name *origin">
@@ -368,4 +374,117 @@
 		<xacro:kuka_lwr_gazebo name="${name}"/>
 		<xacro:kuka_lwr_transmission name="${name}"/>
+		<!-- fake stuff for damping and set_point -->
+		<joint name="${name}_a1_joint_add_torque" type="revolute">
+			<axis xyz="0 0 1"/>
+			<limit lower="${min_add_torque}" upper="${max_add_torque}" effort="0" velocity="${rate_add_torque}" />
+			<safety_controller soft_lower_limit="${min_add_torque}" soft_upper_limit="${max_add_torque}" k_position="30" k_velocity="30"/>
+			<parent link="${name}_base_link"/>
+			<child link="${name}_1_link_dummy_add_torque"/>
+		</joint>
+		<link name="${name}_1_link_dummy_add_torque"/>
+		<joint name="${name}_a2_joint_add_torque" type="revolute">
+			<axis xyz="0 0 1"/>
+			<limit lower="${min_add_torque}" upper="${max_add_torque}" effort="0" velocity="${rate_add_torque}" />
+			<safety_controller soft_lower_limit="${min_add_torque}" soft_upper_limit="${max_add_torque}" k_position="30" k_velocity="30"/>
+			<parent link="${name}_1_link"/>
+			<child link="${name}_2_link_dummy_add_torque"/>
+		</joint>
+		<link name="${name}_2_link_dummy_add_torque"/>
+		<joint name="${name}_e1_joint_add_torque" type="revolute">
+			<axis xyz="0 0 1"/>
+			<limit lower="${min_add_torque}" upper="${max_add_torque}" effort="0" velocity="${rate_add_torque}" />
+			<safety_controller soft_lower_limit="${min_add_torque}" soft_upper_limit="${max_add_torque}" k_position="30" k_velocity="30"/>
+			<parent link="${name}_2_link"/>
+			<child link="${name}_3_link_dummy_add_torque"/>
+		</joint>
+		<link name="${name}_3_link_dummy_add_torque"/>
+		<joint name="${name}_a3_joint_add_torque" type="revolute">
+			<axis xyz="0 0 1"/>
+			<limit lower="${min_add_torque}" upper="${max_add_torque}" effort="0" velocity="${rate_add_torque}" />
+			<safety_controller soft_lower_limit="${min_add_torque}" soft_upper_limit="${max_add_torque}" k_position="30" k_velocity="30"/>
+			<parent link="${name}_3_link"/>
+			<child link="${name}_4_link_dummy_add_torque"/>
+		</joint>
+		<link name="${name}_4_link_dummy_add_torque"/>
+		<joint name="${name}_a4_joint_add_torque" type="revolute">
+			<axis xyz="0 0 1"/>
+			<limit lower="${min_add_torque}" upper="${max_add_torque}" effort="0" velocity="${rate_add_torque}" />
+			<safety_controller soft_lower_limit="${min_add_torque}" soft_upper_limit="${max_add_torque}" k_position="30" k_velocity="30"/>
+			<parent link="${name}_4_link"/>
+			<child link="${name}_5_link_dummy_add_torque"/>
+		</joint>
+		<link name="${name}_5_link_dummy_add_torque"/>
+		<joint name="${name}_a5_joint_add_torque" type="revolute">
+			<axis xyz="0 0 1"/>
+			<limit lower="${min_add_torque}" upper="${max_add_torque}" effort="0" velocity="${rate_add_torque}" />
+			<safety_controller soft_lower_limit="${min_add_torque}" soft_upper_limit="${max_add_torque}" k_position="30" k_velocity="30"/>
+			<parent link="${name}_5_link"/>
+			<child link="${name}_6_link_dummy_add_torque"/>
+		</joint>
+		<link name="${name}_6_link_dummy_add_torque"/>
+		<joint name="${name}_a6_joint_add_torque" type="revolute">
+			<axis xyz="0 0 1"/>
+			<limit lower="${min_add_torque}" upper="${max_add_torque}" effort="0" velocity="${rate_add_torque}" />
+			<safety_controller soft_lower_limit="${min_add_torque}" soft_upper_limit="${max_add_torque}" k_position="30" k_velocity="30"/>
+			<parent link="${name}_6_link"/>
+			<child link="${name}_7_link_dummy_add_torque"/>
+		</joint>
+		<link name="${name}_7_link_dummy_add_torque"/>
+		<joint name="${name}_a1_joint_damping" type="revolute">
+			<axis xyz="0 0 1"/>
+			<limit lower="${min_damping}" upper="${max_damping}" effort="0" velocity="${rate_damping}" />
+			<safety_controller soft_lower_limit="${min_damping}" soft_upper_limit="${max_damping}" k_position="30" k_velocity="30"/>
+			<parent link="${name}_base_link"/>
+			<child link="${name}_1_link_dummy_damping"/>
+		</joint>
+		<link name="${name}_1_link_dummy_damping"/>
+		<joint name="${name}_a2_joint_damping" type="revolute">
+			<axis xyz="0 0 1"/>
+			<limit lower="${min_damping}" upper="${max_damping}" effort="0" velocity="${rate_damping}" />
+			<safety_controller soft_lower_limit="${min_damping}" soft_upper_limit="${max_damping}" k_position="30" k_velocity="30"/>
+			<parent link="${name}_1_link"/>
+			<child link="${name}_2_link_dummy_damping"/>
+		</joint>
+		<link name="${name}_2_link_dummy_damping"/>
+		<joint name="${name}_e1_joint_damping" type="revolute">
+			<axis xyz="0 0 1"/>
+			<limit lower="${min_damping}" upper="${max_damping}" effort="0" velocity="${rate_damping}" />
+			<safety_controller soft_lower_limit="${min_damping}" soft_upper_limit="${max_damping}" k_position="30" k_velocity="30"/>
+			<parent link="${name}_2_link"/>
+			<child link="${name}_3_link_dummy_damping"/>
+		</joint>
+		<link name="${name}_3_link_dummy_damping"/>
+		<joint name="${name}_a3_joint_damping" type="revolute">
+			<axis xyz="0 0 1"/>
+			<limit lower="${min_damping}" upper="${max_damping}" effort="0" velocity="${rate_damping}" />
+			<safety_controller soft_lower_limit="${min_damping}" soft_upper_limit="${max_damping}" k_position="30" k_velocity="30"/>
+			<parent link="${name}_3_link"/>
+			<child link="${name}_4_link_dummy_damping"/>
+		</joint>
+		<link name="${name}_4_link_dummy_damping"/>
+		<joint name="${name}_a4_joint_damping" type="revolute">
+			<axis xyz="0 0 1"/>
+			<limit lower="${min_damping}" upper="${max_damping}" effort="0" velocity="${rate_damping}" />
+			<safety_controller soft_lower_limit="${min_damping}" soft_upper_limit="${max_damping}" k_position="30" k_velocity="30"/>
+			<parent link="${name}_4_link"/>
+			<child link="${name}_5_link_dummy_damping"/>
+		</joint>
+		<link name="${name}_5_link_dummy_damping"/>
+		<joint name="${name}_a5_joint_damping" type="revolute">
+			<axis xyz="0 0 1"/>
+			<limit lower="${min_damping}" upper="${max_damping}" effort="0" velocity="${rate_damping}" />
+			<safety_controller soft_lower_limit="${min_damping}" soft_upper_limit="${max_damping}" k_position="30" k_velocity="30"/>
+			<parent link="${name}_5_link"/>
+			<child link="${name}_6_link_dummy_damping"/>
+		</joint>
+		<link name="${name}_6_link_dummy_damping"/>
+		<joint name="${name}_a6_joint_damping" type="revolute">
+			<axis xyz="0 0 1"/>
+			<limit lower="${min_damping}" upper="${max_damping}" effort="0" velocity="${rate_damping}" />
+			<safety_controller soft_lower_limit="${min_damping}" soft_upper_limit="${max_damping}" k_position="30" k_velocity="30"/>
+			<parent link="${name}_6_link"/>
+			<child link="${name}_7_link_dummy_damping"/>
+		</joint>
+		<link name="${name}_7_link_dummy_damping"/>
 	</xacro:macro>
 </robot>

Commit message: Additional interfaces are now in a separate file loaded using true in the property use_extra_joints (default=true) Stiffness, damping and additional_torque limits come now from the manual.

File: lwr_description/model/kuka_lwr.urdf.xacro (robot description, xacro)
@@ -3,9 +3,9 @@
 	<!-- utils /-->
 	<xacro:include filename="$(find lwr_description)/model/utils.xacro"/>
-	<xacro:include filename="$(find lwr_description)/model/kuka_materials.xacro"
-	/>
+	<xacro:include filename="$(find lwr_description)/model/kuka_materials.xacro"/>
 	<!-- gazebo and transmission models /-->
 	<xacro:include filename="$(find lwr_description)/model/kuka_lwr.gazebo.xacro"/>
 	<xacro:include filename="$(find lwr_description)/model/kuka_lwr.transmission.xacro"/>
+	<xacro:include filename="$(find lwr_description)/model/kuka_lwr.stiffness_damping_addtorque.xacro"/>
 	<!-- properties /-->
 	<xacro:property name="base_mass" value="2.0"/>
@@ -15,15 +15,7 @@
 	<xacro:property name="velocity_scale" value="1"/>
 	<xacro:property name="effort_scale" value="1"/>
-	<xacro:property name="max_stiffness" value="5000"/>
-	<xacro:property name="min_stiffness" value="0"/>
-	<xacro:property name="rate_stiffness" value="20000"/> <!-- reflex to stiffness -->
-	<xacro:property name="max_damping" value="1.0"/>
-	<xacro:property name="min_damping" value="0.0"/>
-	<xacro:property name="rate_damping" value="4.0"/> <!-- reflex to damping -->
-	<xacro:property name="max_add_torque" value="-1.0"/>
-	<xacro:property name="min_add_torque" value="1.0"/>
-	<xacro:property name="rate_add_torque" value="8.0"/> <!-- reflex to additional torque -->
+	<xacro:property name="use_extra_joints_default" value="true"/>
 	<!-- URDF model /-->
-	<xacro:macro name="kuka_lwr" params="parent name *origin">
+	<xacro:macro name="kuka_lwr" params="parent name *origin use_extra_joints:=${use_extra_joints_default}">
 		<!-- First (shoulder) element of the arm. Fixed to its parent. -->
 		<joint name="${parent}_${name}_base_joint" type="fixed">
@@ -62,12 +54,4 @@
 			<child link="${name}_1_link"/>
 		</joint>
-		<joint name="${name}_a1_joint_stiffness" type="revolute">
-			<axis xyz="0 0 1"/>
-			<limit lower="${min_stiffness}" upper="${max_stiffness}" effort="0" velocity="${rate_stiffness}" />
-			<safety_controller soft_lower_limit="${min_stiffness}" soft_upper_limit="${max_stiffness}" k_position="30" k_velocity="30"/>
-			<parent link="${name}_base_link"/>
-			<child link="${name}_1_link_dummy"/>
-		</joint>
-		<link name="${name}_1_link_dummy"/>
 		<link name="${name}_1_link">
 			<inertial>
@@ -111,12 +95,4 @@
 			<child link="${name}_2_link"/>
 		</joint>
-		<joint name="${name}_a2_joint_stiffness" type="revolute">
-			<axis xyz="0 0 1"/>
-			<limit lower="${min_stiffness}" upper="${max_stiffness}" effort="0" velocity="${rate_stiffness}" />
-			<safety_controller soft_lower_limit="${min_stiffness}" soft_upper_limit="${max_stiffness}" k_position="30" k_velocity="30"/>
-			<parent link="${name}_1_link"/>
-			<child link="${name}_2_link_dummy"/>
-		</joint>
-		<link name="${name}_2_link_dummy"/>
 		<link name="${name}_2_link">
 			<inertial>
@@ -160,12 +136,4 @@
 			<child link="${name}_3_link"/>
 		</joint>
-		<joint name="${name}_e1_joint_stiffness" type="revolute">
-			<axis xyz="0 0 1"/>
-			<limit lower="${min_stiffness}" upper="${max_stiffness}" effort="0" velocity="${rate_stiffness}" />
-			<safety_controller soft_lower_limit="${min_stiffness}" soft_upper_limit="${max_stiffness}" k_position="30" k_velocity="30"/>
-			<parent link="${name}_2_link"/>
-			<child link="${name}_3_link_dummy"/>
-		</joint>
-		<link name="${name}_3_link_dummy"/>
 		<link name="${name}_3_link">
 			<inertial>
@@ -209,12 +177,4 @@
 			<child link="${name}_4_link"/>
 		</joint>
-		<joint name="${name}_a3_joint_stiffness" type="revolute">
-			<axis xyz="0 0 1"/>
-			<limit lower="${min_stiffness}" upper="${max_stiffness}" effort="0" velocity="${rate_stiffness}" />
-			<safety_controller soft_lower_limit="${min_stiffness}" soft_upper_limit="${max_stiffness}" k_position="30" k_velocity="30"/>
-			<parent link="${name}_3_link"/>
-			<child link="${name}_4_link_dummy"/>
-		</joint>
-		<link name="${name}_4_link_dummy"/>
 		<link name="${name}_4_link">
 			<inertial>
@@ -258,12 +218,4 @@
 			<child link="${name}_5_link"/>
 		</joint>
-		<joint name="${name}_a4_joint_stiffness" type="revolute">
-			<axis xyz="0 0 1"/>
-			<limit lower="${min_stiffness}" upper="${max_stiffness}" effort="0" velocity="${rate_stiffness}" />
-			<safety_controller soft_lower_limit="${min_stiffness}" soft_upper_limit="${max_stiffness}" k_position="30" k_velocity="30"/>
-			<parent link="${name}_4_link"/>
-			<child link="${name}_5_link_dummy"/>
-		</joint>
-		<link name="${name}_5_link_dummy"/>
 		<link name="${name}_5_link">
 			<inertial>
@@ -307,12 +259,4 @@
 			<child link="${name}_6_link"/>
 		</joint>
-		<joint name="${name}_a5_joint_stiffness" type="revolute">
-			<axis xyz="0 0 1"/>
-			<limit lower="${min_stiffness}" upper="${max_stiffness}" effort="0" velocity="${rate_stiffness}" />
-			<safety_controller soft_lower_limit="${min_stiffness}" soft_upper_limit="${max_stiffness}" k_position="30" k_velocity="30"/>
-			<parent link="${name}_5_link"/>
-			<child link="${name}_6_link_dummy"/>
-		</joint>
-		<link name="${name}_6_link_dummy"/>
 		<link name="${name}_6_link">
 			<inertial>
@@ -344,12 +288,4 @@
 			<child link="${name}_7_link"/>
 		</joint>
-		<joint name="${name}_a6_joint_stiffness" type="revolute">
-			<axis xyz="0 0 1"/>
-			<limit lower="${min_stiffness}" upper="${max_stiffness}" effort="0" velocity="${rate_stiffness}" />
-			<safety_controller soft_lower_limit="${min_stiffness}" soft_upper_limit="${max_stiffness}" k_position="30" k_velocity="30"/>
-			<parent link="${name}_6_link"/>
-			<child link="${name}_7_link_dummy"/>
-		</joint>
-		<link name="${name}_7_link_dummy"/>
 		<link name="${name}_7_link">
 			<inertial>
@@ -374,117 +310,7 @@
 		<xacro:kuka_lwr_gazebo name="${name}"/>
 		<xacro:kuka_lwr_transmission name="${name}"/>
-		<!-- fake stuff for damping and set_point -->
-		<joint name="${name}_a1_joint_add_torque" type="revolute">
-			<axis xyz="0 0 1"/>
-			<limit lower="${min_add_torque}" upper="${max_add_torque}" effort="0" velocity="${rate_add_torque}" />
-			<safety_controller soft_lower_limit="${min_add_torque}" soft_upper_limit="${max_add_torque}" k_position="30" k_velocity="30"/>
-			<parent link="${name}_base_link"/>
-			<child link="${name}_1_link_dummy_add_torque"/>
-		</joint>
-		<link name="${name}_1_link_dummy_add_torque"/>
-		<joint name="${name}_a2_joint_add_torque" type="revolute">
-			<axis xyz="0 0 1"/>
-			<limit lower="${min_add_torque}" upper="${max_add_torque}" effort="0" velocity="${rate_add_torque}" />
-			<safety_controller soft_lower_limit="${min_add_torque}" soft_upper_limit="${max_add_torque}" k_position="30" k_velocity="30"/>
-			<parent link="${name}_1_link"/>
-			<child link="${name}_2_link_dummy_add_torque"/>
-		</joint>
-		<link name="${name}_2_link_dummy_add_torque"/>
-		<joint name="${name}_e1_joint_add_torque" type="revolute">
-			<axis xyz="0 0 1"/>
-			<limit lower="${min_add_torque}" upper="${max_add_torque}" effort="0" velocity="${rate_add_torque}" />
-			<safety_controller soft_lower_limit="${min_add_torque}" soft_upper_limit="${max_add_torque}" k_position="30" k_velocity="30"/>
-			<parent link="${name}_2_link"/>
-			<child link="${name}_3_link_dummy_add_torque"/>
-		</joint>
-		<link name="${name}_3_link_dummy_add_torque"/>
-		<joint name="${name}_a3_joint_add_torque" type="revolute">
-			<axis xyz="0 0 1"/>
-			<limit lower="${min_add_torque}" upper="${max_add_torque}" effort="0" velocity="${rate_add_torque}" />
-			<safety_controller soft_lower_limit="${min_add_torque}" soft_upper_limit="${max_add_torque}" k_position="30" k_velocity="30"/>
-			<parent link="${name}_3_link"/>
-			<child link="${name}_4_link_dummy_add_torque"/>
-		</joint>
-		<link name="${name}_4_link_dummy_add_torque"/>
-		<joint name="${name}_a4_joint_add_torque" type="revolute">
-			<axis xyz="0 0 1"/>
-			<limit lower="${min_add_torque}" upper="${max_add_torque}" effort="0" velocity="${rate_add_torque}" />
-			<safety_controller soft_lower_limit="${min_add_torque}" soft_upper_limit="${max_add_torque}" k_position="30" k_velocity="30"/>
-			<parent link="${name}_4_link"/>
-			<child link="${name}_5_link_dummy_add_torque"/>
-		</joint>
-		<link name="${name}_5_link_dummy_add_torque"/>
-		<joint name="${name}_a5_joint_add_torque" type="revolute">
-			<axis xyz="0 0 1"/>
-			<limit lower="${min_add_torque}" upper="${max_add_torque}" effort="0" velocity="${rate_add_torque}" />
-			<safety_controller soft_lower_limit="${min_add_torque}" soft_upper_limit="${max_add_torque}" k_position="30" k_velocity="30"/>
-			<parent link="${name}_5_link"/>
-			<child link="${name}_6_link_dummy_add_torque"/>
-		</joint>
-		<link name="${name}_6_link_dummy_add_torque"/>
-		<joint name="${name}_a6_joint_add_torque" type="revolute">
-			<axis xyz="0 0 1"/>
-			<limit lower="${min_add_torque}" upper="${max_add_torque}" effort="0" velocity="${rate_add_torque}" />
-			<safety_controller soft_lower_limit="${min_add_torque}" soft_upper_limit="${max_add_torque}" k_position="30" k_velocity="30"/>
-			<parent link="${name}_6_link"/>
-			<child link="${name}_7_link_dummy_add_torque"/>
-		</joint>
-		<link name="${name}_7_link_dummy_add_torque"/>
-		<joint name="${name}_a1_joint_damping" type="revolute">
-			<axis xyz="0 0 1"/>
-			<limit lower="${min_damping}" upper="${max_damping}" effort="0" velocity="${rate_damping}" />
-			<safety_controller soft_lower_limit="${min_damping}" soft_upper_limit="${max_damping}" k_position="30" k_velocity="30"/>
-			<parent link="${name}_base_link"/>
-			<child link="${name}_1_link_dummy_damping"/>
-		</joint>
-		<link name="${name}_1_link_dummy_damping"/>
-		<joint name="${name}_a2_joint_damping" type="revolute">
-			<axis xyz="0 0 1"/>
-			<limit lower="${min_damping}" upper="${max_damping}" effort="0" velocity="${rate_damping}" />
-			<safety_controller soft_lower_limit="${min_damping}" soft_upper_limit="${max_damping}" k_position="30" k_velocity="30"/>
-			<parent link="${name}_1_link"/>
-			<child link="${name}_2_link_dummy_damping"/>
-		</joint>
-		<link name="${name}_2_link_dummy_damping"/>
-		<joint name="${name}_e1_joint_damping" type="revolute">
-			<axis xyz="0 0 1"/>
-			<limit lower="${min_damping}" upper="${max_damping}" effort="0" velocity="${rate_damping}" />
-			<safety_controller soft_lower_limit="${min_damping}" soft_upper_limit="${max_damping}" k_position="30" k_velocity="30"/>
-			<parent link="${name}_2_link"/>
-			<child link="${name}_3_link_dummy_damping"/>
-		</joint>
-		<link name="${name}_3_link_dummy_damping"/>
-		<joint name="${name}_a3_joint_damping" type="revolute">
-			<axis xyz="0 0 1"/>
-			<limit lower="${min_damping}" upper="${max_damping}" effort="0" velocity="${rate_damping}" />
-			<safety_controller soft_lower_limit="${min_damping}" soft_upper_limit="${max_damping}" k_position="30" k_velocity="30"/>
-			<parent link="${name}_3_link"/>
-			<child link="${name}_4_link_dummy_damping"/>
-		</joint>
-		<link name="${name}_4_link_dummy_damping"/>
-		<joint name="${name}_a4_joint_damping" type="revolute">
-			<axis xyz="0 0 1"/>
-			<limit lower="${min_damping}" upper="${max_damping}" effort="0" velocity="${rate_damping}" />
-			<safety_controller soft_lower_limit="${min_damping}" soft_upper_limit="${max_damping}" k_position="30" k_velocity="30"/>
-			<parent link="${name}_4_link"/>
-			<child link="${name}_5_link_dummy_damping"/>
-		</joint>
-		<link name="${name}_5_link_dummy_damping"/>
-		<joint name="${name}_a5_joint_damping" type="revolute">
-			<axis xyz="0 0 1"/>
-			<limit lower="${min_damping}" upper="${max_damping}" effort="0" velocity="${rate_damping}" />
-			<safety_controller soft_lower_limit="${min_damping}" soft_upper_limit="${max_damping}" k_position="30" k_velocity="30"/>
-			<parent link="${name}_5_link"/>
-			<child link="${name}_6_link_dummy_damping"/>
-		</joint>
-		<link name="${name}_6_link_dummy_damping"/>
-		<joint name="${name}_a6_joint_damping" type="revolute">
-			<axis xyz="0 0 1"/>
-			<limit lower="${min_damping}" upper="${max_damping}" effort="0" velocity="${rate_damping}" />
-			<safety_controller soft_lower_limit="${min_damping}" soft_upper_limit="${max_damping}" k_position="30" k_velocity="30"/>
-			<parent link="${name}_6_link"/>
-			<child link="${name}_7_link_dummy_damping"/>
-		</joint>
-		<link name="${name}_7_link_dummy_damping"/>
+		<xacro:if value = "${use_extra_joints}">
+			<xacro:kuka_lwr_stiffness_damping_addtorque name="${name}"/>
+		</xacro:if>
 	</xacro:macro>
 </robot>

Commit message: - temporarily remove friction and damping in the urdf in order to properly invert the dynamics

File: lwr_description/model/kuka_lwr.urdf.xacro (robot description, xacro)
@@ -52,5 +52,5 @@
 			<axis xyz="0 0 1"/>
 			<limit lower="${-170 * M_PI / 180}" upper="${170 * M_PI / 180}" effort="176" velocity="${velocity_scale * 110 * M_PI / 180}" />
-			<dynamics friction="10.0" damping="1.0"/>
+			<dynamics friction="0.0" damping="0.0"/>
 			<parent link="${name}_base_link"/>
 			<child link="${name}_1_link"/>
@@ -101,5 +101,5 @@
 			<axis xyz="0 -1 0"/>
 			<limit lower="${-120 * M_PI / 180}" upper="${120 * M_PI / 180}" effort="176" velocity="${velocity_scale * 110 * M_PI / 180}" />
-			<dynamics friction="10.0" damping="1.0"/>
+			<dynamics friction="0.0" damping="0.0"/>
 			<parent link="${name}_1_link"/>
 			<child link="${name}_2_link"/>
@@ -150,5 +150,5 @@
 			<axis xyz="0 0 1"/>
 			<limit lower="${-170 * M_PI / 180}" upper="${170 * M_PI / 180}" effort="100" velocity="${velocity_scale * 128 * M_PI / 180}" />
-			<dynamics friction="10.0" damping="1.0"/>
+			<dynamics friction="0.0" damping="0.0"/>
 			<parent link="${name}_2_link"/>
 			<child link="${name}_3_link"/>
@@ -199,5 +199,5 @@
 			<axis xyz="0 1 0"/>
 			<limit lower="${-120 * M_PI / 180}" upper="${120 * M_PI / 180}" effort="100" velocity="${velocity_scale * 128 * M_PI / 180}" />
-			<dynamics friction="10.0" damping="1.0"/>
+			<dynamics friction="0.0" damping="0.0"/>
 			<parent link="${name}_3_link"/>
 			<child link="${name}_4_link"/>
@@ -248,5 +248,5 @@
 			<axis xyz="0 0 1"/>
 			<limit lower="${-170 * M_PI / 180}" upper="${170 * M_PI / 180}" effort="100" velocity="${velocity_scale * 204 * M_PI / 180}" />
-			<dynamics friction="10.0" damping="1.0"/>
+			<dynamics friction="0.0" damping="0.0"/>
 			<parent link="${name}_4_link"/>
 			<child link="${name}_5_link"/>
@@ -297,5 +297,5 @@
 			<axis xyz="0 -1 0"/>
 			<limit lower="${-120 * M_PI / 180}" upper="${120 * M_PI / 180}" effort="38" velocity="${velocity_scale * 184 * M_PI / 180}" />
-			<dynamics friction="10.0" damping="1.0"/>
+			<dynamics friction="0.0" damping="0.0"/>
 			<parent link="${name}_5_link"/>
 			<child link="${name}_6_link"/>
@@ -334,5 +334,5 @@
 			<axis xyz="0 0 1"/>
 			<limit lower="${-170 * M_PI / 180}" upper="${170 * M_PI / 180}" effort="38" velocity="${velocity_scale * 184 * M_PI / 180}" />
-			<dynamics friction="10.0" damping="1.0"/>
+			<dynamics friction="0.0" damping="0.0"/>
 			<parent link="${name}_6_link"/>
 			<child link="${name}_7_link"/>
