Commit message: Change mass of the sensor body to a smaller value

File: lwr_description/model/kuka_lwr.urdf.xacro (robot description, xacro)
@@ -373,7 +373,7 @@
 		<link name="end_effector">
 			<inertial>
-				<mass value="0.1"/>
+				<mass value="0.00001"/>
 				<origin xyz="0 0 0"/>
-				<cylinder_inertia_def radius="0.03" length="0.01" mass="0.1"/>
+				<cylinder_inertia_def radius="0.03" length="0.01" mass="0.00001"/>
 			</inertial>
 			<visual>

Commit message: move the end effector frame so that it concides with the previous link frame. It is required to simulate sensing of wrenches with a reference point on the tip of the 7th link.

File: lwr_description/model/kuka_lwr.urdf.xacro (robot description, xacro)
@@ -367,5 +367,5 @@
 		</link>
 		<joint name="sensor_joint" type="fixed">
-			<origin xyz="0 0 0.005" rpy="0 0 0"/>
+			<origin xyz="0 0 0" rpy="0 0 0"/>
 			<parent link="${name}_7_link"/>
 			<child link="end_effector"/>
@@ -374,9 +374,9 @@
 			<inertial>
 				<mass value="0.00001"/>
-				<origin xyz="0 0 0"/>
+				<origin xyz="0 0 0.005"/>
 				<cylinder_inertia_def radius="0.03" length="0.01" mass="0.00001"/>
 			</inertial>
 			<visual>
-				<origin xyz="0 0 0" rpy="0 0 0"/>
+				<origin xyz="0 0 0.005" rpy="0 0 0"/>
 				<geometry>
 				  <cylinder radius="0.03" length="0.01"/>
@@ -385,5 +385,5 @@
 			</visual>
 			<collision>
-			<origin xyz="0 0 0" rpy="0 0 0"/>
+			<origin xyz="0 0 0.005" rpy="0 0 0"/>
 			<geometry>
 				<cylinder radius="0.03" length="0.01"/>

Commit message: change the end effector shape to obtain a stable force measurement

File: lwr_description/model/kuka_lwr.urdf.xacro (robot description, xacro)
@@ -378,15 +378,28 @@
 			</inertial>
 			<visual>
-				<origin xyz="0 0 0.005" rpy="0 0 0"/>
-				<geometry>
-				  <cylinder radius="0.03" length="0.01"/>
-				</geometry>
-			<material name="Black"/>
-			</visual>
-			<collision>
-			<origin xyz="0 0 0.005" rpy="0 0 0"/>
+				<origin xyz="0 0 0.01" rpy="0 0 0"/>
+				<geometry>
+				  <cylinder radius="0.03" length="0.02"/>
+				</geometry>
+			<material name="Red"/>
+			</visual>
+			<visual>
+				<origin xyz="0 0 0.02" rpy="0 0 0"/>
+				<geometry>
+				  <sphere radius="0.01" />
+				</geometry>
+			<material name="Red"/>
+			</visual>
+			<collision>
+			<origin xyz="0 0 0.01" rpy="0 0 0"/>
 			<geometry>
-				<cylinder radius="0.03" length="0.01"/>
+				<cylinder radius="0.03" length="0.02"/>
 			</geometry>
+			</collision>
+			<collision>
+				<origin xyz="0 0 0.02" rpy="0 0 0"/>
+				<geometry>
+				  <sphere radius="0.01" />
+				</geometry>
 			</collision>
 		</link>
